Commit message: Added URDF with Eyes and add relative Jacobian

File: share/romeo3FEB2015.urdf (robot description, URDF)
Before this commit: robot romeoH37V1, 24 links, 23 joints
Links:
- removed link LEye
- removed link LEyeYawLink
- removed link REye
- removed link REyeYawLink
Joints:
- removed joint LEyePitch
- removed joint LEyeYaw
- removed joint REyePitch
- removed joint REyeYaw
