Commit message: New version of URDF->October2015

File: share/romeo.urdf (robot description, URDF)
Before this commit: robot romeoH37V1, 24 links, 23 joints
Links:
- removed link HeadPitchLink
- removed link HeadRollLink
- removed link LElbowRollLink
- removed link LElbowYawLink
- removed link LEye
- removed link LEyeYawLink
- removed link LShoulderPitchLink
- removed link LShoulderYawLink
- removed link LWristRollLink
- removed link LWristYawLink
- removed link NeckPitchLink
- removed link NeckYawLink
- removed link RElbowRollLink
- removed link RElbowYawLink
- removed link REye
- removed link REyeYawLink
- removed link RShoulderPitchLink
- removed link RShoulderYawLink
- removed link RWristRollLink
- removed link RWristYawLink
- removed link l_wrist
- removed link r_wrist
- removed link torso
- added link HeadPitch_link, mass 0.158407
- added link HeadRoll_link, mass 2.07047; visual mesh filename=package://romeo/meshes/HeadRoll.mesh scale=1 1 1
- added link LElbowRoll_link, mass 0.600439
- added link LElbowYaw_link, mass 0.460203; visual mesh filename=package://romeo/meshes/LElbowYaw.mesh scale=1 1 1
- added link LEyePitch_link, mass 0.01; visual mesh filename=package://romeo/meshes/LEye.mesh scale=1 1 1
- added link LEyeYaw_link, mass 0.01
- added link LShoulderPitch_link, mass 0.541429
- added link LShoulderYaw_link, mass 0.861545; visual mesh filename=package://romeo/meshes/LShoulderYaw.mesh scale=1 1 1
- added link LWristPitch_link, mass 0.442191; visual mesh filename=package://romeo/meshes/LWristPitch.mesh scale=1 1 1
- added link LWristRoll_link, mass 0.218316; visual mesh filename=package://romeo/meshes/LWristRoll.mesh scale=1 1 1
- added link LWristYaw_link, mass 0.0758774; visual mesh filename=package://romeo/meshes/LWristYaw.mesh scale=1 1 1
- added link NeckPitch_link, mass 0.345282; visual mesh filename=package://romeo/meshes/NeckPitch.mesh scale=1 1 1
- added link NeckYaw_link, mass 0.377845
- added link RElbowRoll_link, mass 0.600439
- added link RElbowYaw_link, mass 0.460203; visual mesh filename=package://romeo/meshes/RElbowYaw.mesh scale=1 1 1
- added link REyePitch_link, mass 0.01; visual mesh filename=package://romeo/meshes/REye.mesh scale=1 1 1
- added link REyeYaw_link, mass 0.01
- added link RShoulderPitch_link, mass 0.541429
- added link RShoulderYaw_link, mass 0.861545; visual mesh filename=package://romeo/meshes/RShoulderYaw.mesh scale=1 1 1
- added link RWristPitch_link, mass 0.442191; visual mesh filename=package://romeo/meshes/RWristPitch.mesh scale=1 1 1
- added link RWristRoll_link, mass 0.218316; visual mesh filename=package://romeo/meshes/RWristRoll.mesh scale=1 1 1
- added link RWristYaw_link, mass 0.0758774; visual mesh filename=package://romeo/meshes/RWristYaw.mesh scale=1 1 1
- added link Torso_link, mass 5.85463; visual mesh filename=package://romeo/meshes/Torso.mesh scale=1 1 1
Joints:
- removed joint HeadPitch
- removed joint HeadRoll
- removed joint LElbowRoll
- removed joint LElbowYaw
- removed joint LEyePitch
- removed joint LEyeYaw
- removed joint LShoulderPitch
- removed joint LShoulderYaw
- removed joint LWristPitch
- removed joint LWristRoll
- removed joint LWristYaw
- removed joint NeckPitch
- removed joint NeckYaw
- removed joint RElbowRoll
- removed joint RElbowYaw
- removed joint REyePitch
- removed joint REyeYaw
- removed joint RShoulderPitch
- removed joint RShoulderYaw
- removed joint RWristPitch
- removed joint RWristRoll
- removed joint RWristYaw
- added joint HeadPitch_joint: type revolute, parent NeckPitch_link, child HeadPitch_link, origin xyz=0 0 0.0951 rpy=0 -0 0, axis 0 1 0, limit lower=-0.2571 upper=0.2971 effort=2.57 velocity=1.9
- added joint HeadRoll_joint: type revolute, parent HeadPitch_link, child HeadRoll_link, origin xyz=0 0 0 rpy=0 -0 0, axis 1 0 0, limit lower=-0.4887 upper=0.4887 effort=3.748 velocity=1.5
- added joint LElbowRoll_joint: type revolute, parent LShoulderYaw_link, child LElbowRoll_link, origin xyz=0.210824 7.40511e-09 -0.008631 rpy=-2.56114e-09 -0 -9.31322e-09, axis 0.998889 0.0139984 0.044995, limit lower=-2.2148 upper=1.9042 effort=7.404 velocity=3.7
- added joint LElbowYaw_joint: type revolute, parent LElbowRoll_link, child LElbowYaw_link, origin xyz=0 0 0 rpy=-1.49504e-08 -1.86264e-08 2.12577e-09, axis -0.0449994 0 0.998987, limit lower=-1.5228 upper=0.0044 effort=6.02 velocity=4
- added joint LEyePitch_joint: type revolute, parent LEyeYaw_link, child LEyePitch_link, origin xyz=0 0 0 rpy=0 -0 0, axis 0 1 0, limit lower=-0.349066 upper=0.349066 effort=0.01752 velocity=293.215
- added joint LEyeYaw_joint: type revolute, parent HeadRoll_link, child LEyeYaw_link, origin xyz=0.08948 0.03192 0.05425 rpy=0 -0 0, axis 0 0 1, limit lower=-0.523599 upper=0.523599 effort=0.01752 velocity=293.215
- added joint LShoulderPitch_joint: type revolute, parent Torso_link, child LShoulderPitch_link, origin xyz=0.049862 0.19 0.073851 rpy=1.49012e-08 7.45058e-09 0, axis 0.417025 0.895055 -0.15801, limit lower=-1.3491 upper=2.2462 effort=19.095 velocity=2.2
- added joint LShoulderYaw_joint: type revolute, parent LShoulderPitch_link, child LShoulderYaw_link, origin xyz=0 0 0 rpy=2.98023e-08 1.11759e-08 -5.58793e-08, axis 0.0401398 0.155542 0.987013, limit lower=-0.5768 upper=0.9242 effort=9.031 velocity=4
- added joint LWristPitch_joint: type revolute, parent LWristYaw_link, child LWristPitch_link, origin xyz=0 0 0 rpy=0 -0 0, axis 0 1 0, limit lower=-0.988 upper=0.8969 effort=0.6 velocity=3.75
- added joint LWristRoll_joint: type revolute, parent LElbowYaw_link, child LWristRoll_link, origin xyz=0.190404 -4.65661e-10 0.008631 rpy=1.6234e-11 -7.45058e-09 9.32998e-10, axis 0.998987 0 0.0449994, limit lower=-3.6303 upper=0.4887 effort=2.177 velocity=1.1
- added joint LWristYaw_joint: type revolute, parent LWristRoll_link, child LWristYaw_link, origin xyz=0 0 0 rpy=0 -0 0, axis -0.0449994 0 0.998987, limit lower=-0.4014 upper=0.4014 effort=0.862 velocity=2.26
- added joint NeckPitch_joint: type revolute, parent NeckYaw_link, child NeckPitch_link, origin xyz=0 0 0 rpy=0 -2.98023e-08 0, axis 0 1 0, limit lower=-0.3142 upper=0.6632 effort=5.956 velocity=2.2
- added joint NeckYaw_joint: type revolute, parent Torso_link, child NeckYaw_link, origin xyz=0.0548 0 0.1675 rpy=0 -2.98023e-08 0, axis 0.173651 0 0.984807, limit lower=-2.0595 upper=2.0595 effort=7.324 velocity=4
- added joint RElbowRoll_joint: type revolute, parent RShoulderYaw_link, child RElbowRoll_link, origin xyz=0.210824 -1.48548e-08 -0.008631 rpy=6.69388e-09 7.45058e-09 -7.91624e-08, axis 0.998889 -0.0139984 0.044995, limit lower=-1.9047 upper=2.2143 effort=7.404 velocity=3.7
- added joint RElbowYaw_joint: type revolute, parent RElbowRoll_link, child RElbowYaw_link, origin xyz=0 0 0 rpy=1.49504e-08 -1.86264e-08 -2.12577e-09, axis -0.0449994 0 0.998987, limit lower=-0.0047 upper=1.5225 effort=6.02 velocity=4
- added joint REyePitch_joint: type revolute, parent REyeYaw_link, child REyePitch_link, origin xyz=0 0 0 rpy=0 -0 0, axis 0 1 0, limit lower=-0.349066 upper=0.349066 effort=0.01752 velocity=293.215
- added joint REyeYaw_joint: type revolute, parent HeadRoll_link, child REyeYaw_link, origin xyz=0.08948 -0.03192 0.05425 rpy=0 -0 0, axis 0 0 1, limit lower=-0.523599 upper=0.523599 effort=0.01752 velocity=293.215
- added joint RShoulderPitch_joint: type revolute, parent Torso_link, child RShoulderPitch_link, origin xyz=0.049862 -0.19 0.073851 rpy=-1.49012e-08 7.45058e-09 0, axis -0.417025 0.895055 0.15801, limit lower=-1.4554 upper=2.1399 effort=19.095 velocity=2.2
- added joint RShoulderYaw_joint: type revolute, parent RShoulderPitch_link, child RShoulderYaw_link, origin xyz=0 0 0 rpy=-2.98023e-08 1.49012e-08 -6.42613e-08, axis 0.0401398 -0.155542 0.987014, limit lower=-1.0985 upper=0.4025 effort=9.031 velocity=4
- added joint RWristPitch_joint: type revolute, parent RWristYaw_link, child RWristPitch_link, origin xyz=0 0 0 rpy=0 -0 0, axis 0 1 0, limit lower=-0.9868 upper=0.8981 effort=0.6 velocity=3.75
- added joint RWristRoll_joint: type revolute, parent RElbowYaw_link, child RWristRoll_link, origin xyz=0.190404 4.65661e-10 0.008631 rpy=-1.6234e-11 -7.45058e-09 -9.32998e-10, axis 0.998987 0 0.0449994, limit lower=-0.4887 upper=3.6303 effort=2.177 velocity=1.1
- added joint RWristYaw_joint: type revolute, parent RWristRoll_link, child RWristYaw_link, origin xyz=0 0 0 rpy=0 -0 0, axis -0.0449994 0 0.998987, limit lower=-0.4014 upper=0.4014 effort=0.862 velocity=2.26
- joint base_joint: child torso -> Torso_link

Commit message: Added Trunk to Model, added get Jacobian from trunk to Leye, compatible with last version of visp

File: share/romeo.urdf (robot description, URDF)
Before this commit: robot RomeoH37, 24 links, 23 joints
Links:
- added link TrunkYaw_link
Joints:
- added joint TrunkYaw_joint: type revolute, parent TrunkYaw_link, child Torso_link, origin xyz=-0.0499 0 1.0146  rpy=0.0 0.0 0.0, axis 0 0 -1, limit lower=-0.7575 upper=0.7575 effort=28.021 velocity=1.5
- joint base_joint: child Torso_link -> TrunkYaw_link
